File: pcb/MicroMacroPad.kicad_sch (KiCad schematic)
At the start: 38 parts, among them J1 Conn_01x04_Pin, SW1 SW_Push, SW10 SW_Push, SW11 SW_Push, SW12 SW_Push, SW2 SW_Push, SW3 SW_Push, SW4 SW_Push, SW5 SW_Push, SW6 SW_Push, SW7 SW_Push, SW8 SW_Push, SW9 SW_Push, U1 XIAO-RP2040-DIP

Commit message: V2 upload
Parts:
- D13, D14, D15, D16, D17, D18, D19, D20, D21, D22, D23, D24: footprint kicad-footprint:LED_SK6812MINI -> footprints:LED_SK6812MINI
- J1: footprint kicad-footprint:SSD1306-0.91-OLED-4pin-128x32 -> footprints:SSD1306-0.91-OLED-4pin-128x32
- U1: footprint kicad-footprint:XIAO-RP2040-DIP -> footprints:XIAO-RP2040-DIP
Connections:
- net row0 is gone; now on net col1: SW1.2, SW10.2, SW4.2, SW7.2, U1.8 (GPIO1/RX)
- net +5V: no longer J1.2 (Pin_2)
- net col1: no longer D4.1 (K), D5.1 (K), D6.1 (K), U1.1 (GPIO26/ADC0/A0)
- net col2: now also D10.1 (K), D11.1 (K), D12.1 (K), D7.1 (K), D8.1 (K), D9.1 (K), SW11.2, SW12.2, SW2.2, SW3.2, SW5.2, SW6.2, SW8.2, SW9.2, U1.1 (GPIO26/ADC0/A0), U1.10 (GPIO4/MISO), U1.4 (GPIO29/ADC3/A3), U1.9 (GPIO2/SCK); no longer D1.1 (K), D2.1 (K), D3.1 (K), U1.2 (GPIO27/ADC1/A1)
- net at D18.4 (DIN): now also D15.2 (DOUT); no longer D19.4 (DIN)
- net at D16.2 (DOUT): now also D19.4 (DIN); no longer D15.2 (DOUT)
- net at D24.4 (DIN): now also D21.2 (DOUT)
- net +3V3: now reaches U1.12 (3V3)
- net +3V3: now also J1.2 (Pin_2)
- net at D22.2 (DOUT): no longer D21.2 (DOUT)
- removed net col0: D10.1 (K), D11.1 (K), D12.1 (K), D7.1 (K), D8.1 (K), D9.1 (K), SW11.2, SW12.2, SW2.2, SW3.2, SW5.2, SW6.2, SW8.2, SW9.2, U1.10 (GPIO4/MISO), U1.3 (GPIO28/ADC2/A2), U1.4 (GPIO29/ADC3/A3), U1.9 (GPIO2/SCK)
- new net row2: D1.1 (K), D2.1 (K), D3.1 (K), U1.2 (GPIO27/ADC1/A1)
- new net row3: D4.1 (K), D5.1 (K), D6.1 (K), U1.3 (GPIO28/ADC2/A2)
